File: pcb/kicad5.kicad_sch (KiCad schematic)
At the start: 8 parts, among them SW1 SW_Push, SW2 SW_Push, SW3 SW_Push, SW4 SW_Push, SW5 RotaryEncoder_Switch, U1 XIAO-RP2040-DIP

Commit message: chnges
Parts:
- added D3, D4: SK6812MINI, LED_SMD:LED_SK6812MINI_PLCC4_3.5x3.5mm_P1.75mm, symbol LED:SK6812MINI
- added U2: SSD1306, Oled:SSD1306-0.91-OLED-4pin-128x32, symbol OLED:SSD1306
Connections:
- net +5V: now also D1.4 (VDD), D2.4 (VDD), D3.4 (VDD), D4.4 (VDD)
- net GND: now also D3.2 (VSS), D4.2 (VSS), U2.9 (GND); no longer D1.4 (VDD), D2.4 (VDD)
- net at D2.1 (DOUT): now also D3.3 (DIN)
- net at D1.3 (DIN): now also U1.4 (GPIO29/ADC3/A3); no longer U1.5 (GPIO6/SDA)
- net +3.3V: now reaches U1.12 (3V3)
- net +3.3V: now also U2.10 (VCC)
- net at U1.6 (GPIO7/SCL): now also U2.11 (SCL)
- new net: D3.1 (DOUT), D4.3 (DIN)
- new net: U1.5 (GPIO6/SDA), U2.12 (SDA)
